Commit message: separate frame and mesh config package

File: chin_description/urdf/chin_arm_frame.urdf.xacro (robot description, xacro)
@@ -132,18 +132,18 @@
   </xacro:macro>
   <!--fixed link0-->
-  <xacro:link_with_sc name="link0" link_height="${link_base_height}" link_radius="${link_base_radius}" pos_xyz="0 0 ${0.5*link_base_height}" visual_color="black" gazebo="${gazebo}">
+  <xacro:link_with_sc name="link_0" link_height="${link_base_height}" link_radius="${link_base_radius}" pos_xyz="0 0 ${0.5*link_base_height}" visual_color="black" gazebo="${gazebo}">
     <self_collision_geometries/>
   </xacro:link_with_sc>
   <!--link1 to link0-->
-  <xacro:link_with_sc name="link1" link_height="${link_1_height}" link_radius="${link_1_radius}" pos_xyz="0 0 ${0.5*link_1_height}" visual_color="silver" gazebo="${gazebo}">
+  <xacro:link_with_sc name="link_1" link_height="${link_1_height}" link_radius="${link_1_radius}" pos_xyz="0 0 ${0.5*link_1_height}" visual_color="silver" gazebo="${gazebo}">
     <self_collision_geometries>
       <xacro:collision_capsule xyz="0 0 ${0.5*link_1_height}" radius="${link_1_radius+safety_distance}" length="${link_1_height+safety_distance}"/>
     </self_collision_geometries>
   </xacro:link_with_sc>
-  <joint name="${arm_id}_joint1" type="revolute">
+  <joint name="${arm_id}_joint_1" type="revolute">
     <safety_controller k_position="100.0" k_velocity="40.0" soft_lower_limit="-${pi}" soft_upper_limit="${pi}"/>
     <origin rpy="0 0 0" xyz="0 0 ${link_base_height}"/>
-    <parent link="${arm_id}_link0"/>
-    <child link="${arm_id}_link1"/>
+    <parent link="${arm_id}_link_0"/>
+    <child link="${arm_id}_link_1"/>
     <axis xyz="0 0 1"/>
     <limit lower="-${pi}" upper="${pi}" effort="0" velocity="0"/>
@@ -151,27 +151,27 @@
   </joint>
   <!--link2 to link1-->
-  <xacro:link_with_sc name="link2" link_height="${link_2_height}" link_radius="${link_2_radius}" pos_xyz="0 0 ${0.5*link_2_height}" gazebo="${gazebo}">
+  <xacro:link_with_sc name="link_2" link_height="${link_2_height}" link_radius="${link_2_radius}" pos_xyz="0 0 ${0.5*link_2_height}" gazebo="${gazebo}">
     <self_collision_geometries>
       <xacro:collision_capsule xyz="0 0 ${0.5*link_2_height}" radius="${link_2_radius+safety_distance}" length="${link_2_height+safety_distance}"/>
     </self_collision_geometries>
   </xacro:link_with_sc>
-  <joint name="${arm_id}_joint2" type="fixed">
+  <joint name="${arm_id}_joint_2" type="fixed">
     <origin rpy="-${0.5*pi} 0 0" xyz="0 0 ${link_1_height}"/>
-    <parent link="${arm_id}_link1"/>
-    <child link="${arm_id}_link2"/>
+    <parent link="${arm_id}_link_1"/>
+    <child link="${arm_id}_link_2"/>
     <axis xyz="0 0 1"/>
     <dynamics D="1" K="7000" damping="0.003" friction="0.0" mu_coulomb="0" mu_viscous="16"/>
   </joint>
   <!--link3 to link2-->
-  <xacro:link_with_sc name="link3" link_height="${link_3_height}" link_radius="${link_3_radius}" pos_xyz="0 0 ${0.5*link_3_height}" visual_color="silver" gazebo="${gazebo}">
+  <xacro:link_with_sc name="link_3" link_height="${link_3_height}" link_radius="${link_3_radius}" pos_xyz="0 0 ${0.5*link_3_height}" visual_color="silver" gazebo="${gazebo}">
     <self_collision_geometries>
       <xacro:collision_capsule xyz="0 0 ${0.5*link_3_height}" radius="${link_3_radius+safety_distance}" length="${link_3_height+safety_distance}"/>
     </self_collision_geometries>
   </xacro:link_with_sc>
-  <joint name="${arm_id}_joint3" type="revolute">
+  <joint name="${arm_id}_joint_3" type="revolute">
     <safety_controller k_position="100.0" k_velocity="40.0" soft_lower_limit="-${pi}" soft_upper_limit="${pi}"/>
     <origin rpy="0 0 0" xyz="0 0 ${link_2_height}"/>
-    <parent link="${arm_id}_link2"/>
-    <child link="${arm_id}_link3"/>
+    <parent link="${arm_id}_link_2"/>
+    <child link="${arm_id}_link_3"/>
     <axis xyz="0 0 1"/>
     <limit lower="-${pi}" upper="${pi}" effort="0" velocity="0"/>
@@ -179,40 +179,40 @@
   </joint>
   <!--link4 to link3-->
-  <xacro:link_with_sc name="link4" link_height="${link_4_height}" link_radius="${link_4_radius}" pos_xyz="0 0 ${0.5*link_4_height}" gazebo="${gazebo}">
+  <xacro:link_with_sc name="link_4" link_height="${link_4_height}" link_radius="${link_4_radius}" pos_xyz="0 0 ${0.5*link_4_height}" gazebo="${gazebo}">
     <self_collision_geometries>
       <xacro:collision_capsule xyz="0 0 ${0.5*link_4_height}" radius="${link_4_radius+safety_distance}" length="${link_4_height+safety_distance}"/>
     </self_collision_geometries>
   </xacro:link_with_sc>
-  <joint name="${arm_id}_joint4" type="fixed">
+  <joint name="${arm_id}_joint_4" type="fixed">
     <origin rpy="${0.5*pi} 0 0" xyz="0 0 ${link_3_height}"/>
-    <parent link="${arm_id}_link3"/>
-    <child link="${arm_id}_link4"/>
+    <parent link="${arm_id}_link_3"/>
+    <child link="${arm_id}_link_4"/>
     <axis xyz="0 0 1"/>
     <dynamics D="1" K="7000" damping="0.003" friction="0.0" mu_coulomb="0" mu_viscous="16"/>
   </joint>
   <!--link5 to link4-->
-  <xacro:link_with_sc name="link5" link_height="${link_5_height}" link_radius="${link_5_radius}" pos_xyz="0 0 ${0.5*link_5_height}" gazebo="${gazebo}">
+  <xacro:link_with_sc name="link_5" link_height="${link_5_height}" link_radius="${link_5_radius}" pos_xyz="0 0 ${0.5*link_5_height}" gazebo="${gazebo}">
     <self_collision_geometries>
       <xacro:collision_capsule xyz="0 0 ${0.5*link_5_height}" radius="${link_5_radius+safety_distance}" length="${link_5_height+safety_distance}"/>
     </self_collision_geometries>
   </xacro:link_with_sc>
-  <joint name="${arm_id}_joint5" type="fixed">
+  <joint name="${arm_id}_joint_5" type="fixed">
     <origin rpy="${0.5*pi} 0 0" xyz="0 0 ${link_4_height}"/>
-    <parent link="${arm_id}_link4"/>
-    <child link="${arm_id}_link5"/>
+    <parent link="${arm_id}_link_4"/>
+    <child link="${arm_id}_link_5"/>
     <axis xyz="0 0 1"/>
     <dynamics D="1" K="7000" damping="0.003" friction="0.0" mu_coulomb="0" mu_viscous="16"/>
   </joint>
   <!--link6 to link5-->
-  <xacro:link_with_sc name="link6" link_height="${link_6_height}" link_radius="${link_6_radius}" pos_xyz="0 0 ${0.5*link_6_height}" visual_color="silver" gazebo="${gazebo}">
+  <xacro:link_with_sc name="link_6" link_height="${link_6_height}" link_radius="${link_6_radius}" pos_xyz="0 0 ${0.5*link_6_height}" visual_color="silver" gazebo="${gazebo}">
     <self_collision_geometries>
       <xacro:collision_capsule xyz="0 0 ${0.5*link_6_height}" radius="${link_6_radius+safety_distance}" length="${link_6_height+safety_distance}"/>
     </self_collision_geometries>
   </xacro:link_with_sc>
-  <joint name="${arm_id}_joint6" type="revolute">
+  <joint name="${arm_id}_joint_6" type="revolute">
     <safety_controller k_position="100.0" k_velocity="40.0" soft_lower_limit="-2.7925" soft_upper_limit="2.7925"/>
     <origin rpy="0 0 0" xyz="0 0 ${link_5_height}"/>
-    <parent link="${arm_id}_link5"/>
-    <child link="${arm_id}_link6"/>
+    <parent link="${arm_id}_link_5"/>
+    <child link="${arm_id}_link_6"/>
     <axis xyz="0 0 1"/>
     <limit lower="-2.7925" upper="2.7925" effort="0" velocity="0"/>
@@ -220,40 +220,40 @@
   </joint>
   <!--link7 to link6-->
-  <xacro:link_with_sc name="link7" link_height="${link_7_height}" link_radius="${link_7_radius}" pos_xyz="0 0 ${0.5*link_7_height}" gazebo="${gazebo}">
+  <xacro:link_with_sc name="link_7" link_height="${link_7_height}" link_radius="${link_7_radius}" pos_xyz="0 0 ${0.5*link_7_height}" gazebo="${gazebo}">
     <self_collision_geometries>
       <xacro:collision_capsule xyz="0 0 ${0.5*link_7_height}" radius="${link_7_radius+safety_distance}" length="${link_7_height+safety_distance}"/>
     </self_collision_geometries>
   </xacro:link_with_sc>
-  <joint name="${arm_id}_joint7" type="fixed">
+  <joint name="${arm_id}_joint_7" type="fixed">
     <origin rpy="-${0.5*pi} 0 0" xyz="0 0 ${link_6_height}"/>
-    <parent link="${arm_id}_link6"/>
-    <child link="${arm_id}_link7"/>
+    <parent link="${arm_id}_link_6"/>
+    <child link="${arm_id}_link_7"/>
     <axis xyz="0 0 1"/>
     <dynamics D="1" K="7000" damping="0.003" friction="0.0" mu_coulomb="0" mu_viscous="16"/>
   </joint>
   <!--link8 to link7-->
-  <xacro:link_with_sc name="link8" link_height="${link_8_height}" link_radius="${link_8_radius}" pos_xyz="0 0 ${0.5*link_8_height}" gazebo="${gazebo}">
+  <xacro:link_with_sc name="link_8" link_height="${link_8_height}" link_radius="${link_8_radius}" pos_xyz="0 0 ${0.5*link_8_height}" gazebo="${gazebo}">
     <self_collision_geometries>
       <xacro:collision_capsule xyz="0 0 ${0.5*link_8_height}" radius="${link_8_radius+safety_distance}" length="${link_8_height+safety_distance}"/>
     </self_collision_geometries>
   </xacro:link_with_sc>
-  <joint name="${arm_id}_joint8" type="fixed">
+  <joint name="${arm_id}_joint_8" type="fixed">
     <origin rpy="-${0.5*pi} 0 0" xyz="0 0 ${link_7_height}"/>
-    <parent link="${arm_id}_link7"/>
-    <child link="${arm_id}_link8"/>
+    <parent link="${arm_id}_link_7"/>
+    <child link="${arm_id}_link_8"/>
     <axis xyz="0 0 1"/>
     <dynamics D="1" K="7000" damping="0.003" friction="0.0" mu_coulomb="0" mu_viscous="16"/>
   </joint>
   <!--link9 to link8-->
-  <xacro:link_with_sc name="link9" link_height="${link_9_height}" link_radius="${link_9_radius}" pos_xyz="0 0 ${0.5*link_9_height}" visual_color="silver" gazebo="${gazebo}">
+  <xacro:link_with_sc name="link_9" link_height="${link_9_height}" link_radius="${link_9_radius}" pos_xyz="0 0 ${0.5*link_9_height}" visual_color="silver" gazebo="${gazebo}">
     <self_collision_geometries>
       <xacro:collision_capsule xyz="0 0 ${0.5*link_9_height}" radius="${link_9_radius+safety_distance}" length="${link_9_height+safety_distance}"/>
     </self_collision_geometries>
   </xacro:link_with_sc>
-  <joint name="${arm_id}_joint9" type="revolute">
+  <joint name="${arm_id}_joint_9" type="revolute">
     <safety_controller k_position="100.0" k_velocity="40.0" soft_lower_limit="-${pi}" soft_upper_limit="${pi}"/>
     <origin rpy="0 0 0" xyz="0 0 ${link_8_height}"/>
-    <parent link="${arm_id}_link8"/>
-    <child link="${arm_id}_link9"/>
+    <parent link="${arm_id}_link_8"/>
+    <child link="${arm_id}_link_9"/>
     <axis xyz="0 0 1"/>
     <limit lower="-${pi}" upper="${pi}" effort="0" velocity="0"/>
@@ -261,27 +261,27 @@
   </joint>
   <!--link10 to link9-->
-  <xacro:link_with_sc name="link10" link_height="${link_10_height}" link_radius="${link_10_radius}" pos_xyz="0 0 ${0.5*link_10_height}" gazebo="${gazebo}">
+  <xacro:link_with_sc name="link_10" link_height="${link_10_height}" link_radius="${link_10_radius}" pos_xyz="0 0 ${0.5*link_10_height}" gazebo="${gazebo}">
     <self_collision_geometries>
       <xacro:collision_capsule xyz="0 0 ${0.5*link_10_height}" radius="${link_10_radius+safety_distance}" length="${link_10_height+safety_distance}"/>
     </self_collision_geometries>
   </xacro:link_with_sc>
-  <joint name="${arm_id}_joint10" type="fixed">
+  <joint name="${arm_id}_joint_10" type="fixed">
     <origin rpy="${0.5*pi} 0 0" xyz="0 0 ${link_9_height}"/>
-    <parent link="${arm_id}_link9"/>
-    <child link="${arm_id}_link10"/>
+    <parent link="${arm_id}_link_9"/>
+    <child link="${arm_id}_link_10"/>
     <axis xyz="0 0 1"/>
     <dynamics D="1" K="7000" damping="0.003" friction="0.0" mu_coulomb="0" mu_viscous="16"/>
   </joint>
   <!--link11 to link10-->
-  <xacro:link_with_sc name="link11" link_height="${link_11_height}" link_radius="${link_11_radius}" pos_xyz="0 0 ${0.5*link_11_height}" visual_color="silver" gazebo="${gazebo}">
+  <xacro:link_with_sc name="link_11" link_height="${link_11_height}" link_radius="${link_11_radius}" pos_xyz="0 0 ${0.5*link_11_height}" visual_color="silver" gazebo="${gazebo}">
     <self_collision_geometries>
       <xacro:collision_capsule xyz="0 0 ${0.5*link_11_height}" radius="${link_11_radius+safety_distance}" length="${link_11_height+safety_distance}"/>
     </self_collision_geometries>
   </xacro:link_with_sc>
-  <joint name="${arm_id}_joint11" type="revolute">
+  <joint name="${arm_id}_joint_11" type="revolute">
     <safety_controller k_position="100.0" k_velocity="40.0" soft_lower_limit="-${pi}" soft_upper_limit="${pi}"/>
     <origin rpy="0 0 0" xyz="0 0 ${link_10_height}"/>
-    <parent link="${arm_id}_link10"/>
-    <child link="${arm_id}_link11"/>
+    <parent link="${arm_id}_link_10"/>
+    <child link="${arm_id}_link_11"/>
     <axis xyz="0 0 1"/>
     <limit lower="-${pi}" upper="${pi}" effort="0" velocity="0"/>
@@ -289,27 +289,27 @@
   </joint>
   <!--link12 to link11-->
-  <xacro:link_with_sc name="link12" link_height="${link_12_height}" link_radius="${link_12_radius}" pos_xyz="0 0 ${0.5*link_12_height}" gazebo="${gazebo}">
+  <xacro:link_with_sc name="link_12" link_height="${link_12_height}" link_radius="${link_12_radius}" pos_xyz="0 0 ${0.5*link_12_height}" gazebo="${gazebo}">
     <self_collision_geometries>
       <xacro:collision_capsule xyz="0 0 ${0.5*link_12_height}" radius="${link_12_radius+safety_distance}" length="${link_12_height+safety_distance}"/>
     </self_collision_geometries>
   </xacro:link_with_sc>
-  <joint name="${arm_id}_joint12" type="fixed">
+  <joint name="${arm_id}_joint_12" type="fixed">
     <origin rpy="-${0.5*pi} 0 0" xyz="0 0 ${link_11_height}"/>
-    <parent link="${arm_id}_link11"/>
-    <child link="${arm_id}_link12"/>
+    <parent link="${arm_id}_link_11"/>
+    <child link="${arm_id}_link_12"/>
     <axis xyz="0 0 1"/>
     <dynamics D="1" K="7000" damping="0.003" friction="0.0" mu_coulomb="0" mu_viscous="16"/>
   </joint>
   <!--link13 to link12-->
-  <xacro:link_with_sc name="link13" link_height="${link_13_height}" link_radius="${link_13_radius}" pos_xyz="0 0 ${0.5*link_13_height}" visual_color="silver" gazebo="${gazebo}">
+  <xacro:link_with_sc name="link_13" link_height="${link_13_height}" link_radius="${link_13_radius}" pos_xyz="0 0 ${0.5*link_13_height}" visual_color="silver" gazebo="${gazebo}">
     <self_collision_geometries>
       <xacro:collision_capsule xyz="0 0 ${0.5*link_13_height}" radius="${link_13_radius+safety_distance}" length="${link_13_height+safety_distance}"/>
     </self_collision_geometries>
   </xacro:link_with_sc>
-  <joint name="${arm_id}_joint13" type="revolute">
+  <joint name="${arm_id}_joint_13" type="revolute">
     <safety_controller k_position="100.0" k_velocity="40.0" soft_lower_limit="-${pi}" soft_upper_limit="${pi}"/>
     <origin rpy="0 0 0" xyz="0 0 ${link_12_height}"/>
-    <parent link="${arm_id}_link12"/>
-    <child link="${arm_id}_link13"/>
+    <parent link="${arm_id}_link_12"/>
+    <child link="${arm_id}_link_13"/>
     <axis xyz="0 0 1"/>
     <limit lower="-${pi}" upper="${pi}" effort="0" velocity="0"/>
@@ -317,9 +317,9 @@
   </joint>
   <!--link14 to link13-->
-  <link name="${arm_id}_link14"/>
-  <joint name="${arm_id}_joint14" type="fixed">
+  <link name="${arm_id}_link_14"/>
+  <joint name="${arm_id}_joint_14" type="fixed">
     <origin rpy="0 0 -${pi}" xyz="0 0 ${link_13_height}"/>
-    <parent link="${arm_id}_link13"/>
-    <child link="${arm_id}_link14"/>
+    <parent link="${arm_id}_link_13"/>
+    <child link="${arm_id}_link_14"/>
   </joint>
 </robot>

File: chin_moveit_config/config/gazebo_chin_arm.urdf (robot description, URDF)
Before this commit: robot chin_arm, 29 links, 28 joints
Links:
- removed link chin_link0
- removed link chin_link0_sc
- removed link chin_link1
- removed link chin_link10
- removed link chin_link10_sc
- removed link chin_link11
- removed link chin_link11_sc
- removed link chin_link12
- removed link chin_link12_sc
- removed link chin_link13
- removed link chin_link13_sc
- removed link chin_link14
- removed link chin_link1_sc
- removed link chin_link2
- removed link chin_link2_sc
- removed link chin_link3
- removed link chin_link3_sc
- removed link chin_link4
- removed link chin_link4_sc
- removed link chin_link5
- removed link chin_link5_sc
- removed link chin_link6
- removed link chin_link6_sc
- removed link chin_link7
- removed link chin_link7_sc
- removed link chin_link8
- removed link chin_link8_sc
- removed link chin_link9
- removed link chin_link9_sc
- added link chin_link_0, mass 0.1; collision mesh filename=package://chin_description/meshes/collision/link_0.stl; visual mesh filename=package://chin_description/meshes/visual/link_0.dae
- added link chin_link_1, mass 0.1; collision mesh filename=package://chin_description/meshes/collision/link_1.stl; visual mesh filename=package://chin_description/meshes/visual/link_1.dae
- added link chin_link_2, mass 0.1; collision mesh filename=package://chin_description/meshes/collision/link_2.stl; visual mesh filename=package://chin_description/meshes/visual/link_2.dae
- added link chin_link_3, mass 0.1; collision mesh filename=package://chin_description/meshes/collision/link_3.stl; visual mesh filename=package://chin_description/meshes/visual/link_3.dae
- added link chin_link_4, mass 0.1; collision mesh filename=package://chin_description/meshes/collision/link_4.stl; visual mesh filename=package://chin_description/meshes/visual/link_4.dae
- added link chin_link_5, mass 0.1; collision mesh filename=package://chin_description/meshes/collision/link_5.stl; visual mesh filename=package://chin_description/meshes/visual/link_5.dae
- added link chin_link_6, mass 0.1; collision mesh filename=package://chin_description/meshes/collision/link_6.stl; visual mesh filename=package://chin_description/meshes/visual/link_6.dae
- added link chin_link_7
Joints:
- removed joint chin_joint1
- removed joint chin_joint10
- removed joint chin_joint11
- removed joint chin_joint12
- removed joint chin_joint13
- removed joint chin_joint14
- removed joint chin_joint2
- removed joint chin_joint3
- removed joint chin_joint4
- removed joint chin_joint5
- removed joint chin_joint6
- removed joint chin_joint7
- removed joint chin_joint8
- removed joint chin_joint9
- removed joint chin_link0_sc_joint
- removed joint chin_link10_sc_joint
- removed joint chin_link11_sc_joint
- removed joint chin_link12_sc_joint
- removed joint chin_link13_sc_joint
- removed joint chin_link1_sc_joint
- removed joint chin_link2_sc_joint
- removed joint chin_link3_sc_joint
- removed joint chin_link4_sc_joint
- removed joint chin_link5_sc_joint
- removed joint chin_link6_sc_joint
- removed joint chin_link7_sc_joint
- removed joint chin_link8_sc_joint
- removed joint chin_link9_sc_joint
- added joint chin_joint_1: type revolute, parent chin_link_0, child chin_link_1, origin xyz=0 0 0.2038 rpy=0 0 0, axis 0 0 1, limit lower=-3.14159265359 upper=3.14159265359 effort=0 velocity=0
- added joint chin_joint_2: type revolute, parent chin_link_1, child chin_link_2, origin xyz=0 0.082 0.081 rpy=-1.57079632679 0 0, axis 0 0 1, limit lower=-3.14159265359 upper=3.14159265359 effort=0 velocity=0
- added joint chin_joint_3: type revolute, parent chin_link_2, child chin_link_3, origin xyz=0 -0.398 0 rpy=3.14159265359 0 0, axis 0 0 1, limit lower=-2.7925 upper=2.7925 effort=0 velocity=0
- added joint chin_joint_4: type revolute, parent chin_link_3, child chin_link_4, origin xyz=0 0.36 -0.02 rpy=3.14159265359 0 0, axis 0 0 1, limit lower=-3.14159265359 upper=3.14159265359 effort=0 velocity=0
- added joint chin_joint_5: type revolute, parent chin_link_4, child chin_link_5, origin xyz=0 -0.083 0.087 rpy=1.57079632679 0 0, axis 0 0 1, limit lower=-3.14159265359 upper=3.14159265359 effort=0 velocity=0
- added joint chin_joint_6: type revolute, parent chin_link_5, child chin_link_6, origin xyz=0 0.083 0.087 rpy=-1.57079632679 0 0, axis 0 0 1, limit lower=-3.14159265359 upper=3.14159265359 effort=0 velocity=0
- added joint chin_joint_7: type fixed, parent chin_link_6, child chin_link_7, origin xyz=0 0 0.077 rpy=0 0 -3.14159265359
