Commit message: revised for collision

File: chin_description/urdf/chin_arm.urdf.xacro (robot description, xacro)
@@ -33,4 +33,5 @@
   <xacro:property name="link_13_height" value="0.077"/>
   <xacro:property name="link_13_radius" value="0.02"/>
+  <xacro:property name="with_mesh" value="false"/>
   <material name="white">
     <color rgba="1 1 1 1"/>
@@ -86,6 +87,10 @@
 	      <origin xyz="${pos_xyz}" rpy="${pos_rpy}"/>
         <geometry>
-          <!--<mesh filename="package://${description_pkg}/meshes/visual/${name}.dae"/>-->
-          <cylinder length="${link_height}" radius="${link_radius}"/>
+          <xacro:if value="${with_mesh == 'true'}">
+            <mesh filename="package://${description_pkg}/meshes/visual/${name}.dae"/>
+          </xacro:if>
+          <xacro:unless value="${with_mesh == 'true'}">
+            <cylinder length="${link_height}" radius="${link_radius}"/>
+          </xacro:unless>
         </geometry>
         <material name="${visual_color}"/>
@@ -94,6 +99,10 @@
 	      <origin xyz="${pos_xyz}" rpy="${pos_rpy}"/>
         <geometry>
-          <!--<mesh filename="package://franka_description/meshes/collision/${name}.stl"/>-->
-          <cylinder length="${link_height}" radius="${link_radius}"/>
+          <xacro:if value="${with_mesh == 'true'}">
+            <mesh filename="package://franka_description/meshes/collision/${name}.stl"/>
+          </xacro:if>
+          <xacro:unless value="${with_mesh == 'true'}">
+            <cylinder length="${link_height}" radius="${link_radius}"/>
+          </xacro:unless>
         </geometry>
       </collision>
@@ -120,5 +129,5 @@
   </xacro:link_with_sc>
   <!--link1 to link0-->
-  <xacro:link_with_sc name="link1" link_height="${link_1_height}" link_radius="${link_1_radius}" pos_xyz="0 0 ${0.5*link_1_height}" pos_rpy="0 0 0" gazebo="${gazebo}">
+  <xacro:link_with_sc name="link1" link_height="${link_1_height}" link_radius="${link_1_radius}" pos_xyz="0 0 ${0.5*link_1_height}" gazebo="${gazebo}">
     <self_collision_geometries>
       <xacro:collision_capsule xyz="0 0 0" radius="${link_1_radius+safety_distance}" length="${link_1_height+safety_distance}"/>
@@ -135,7 +144,7 @@
   </joint>
   <!--link2 to link1-->
-  <xacro:link_with_sc name="link2" link_height="${link_2_height}" link_radius="${link_2_radius}" pos_xyz="0 0 ${0.5*link_2_height}" pos_rpy="0 0 0" gazebo="${gazebo}">
-    <self_collision_geometries>
-      <xacro:collision_capsule xyz="0 0 0" radius="${link_1_radius+safety_distance}" length="${link_1_height+safety_distance}"/>
+  <xacro:link_with_sc name="link2" link_height="${link_2_height}" link_radius="${link_2_radius}" pos_xyz="0 0 ${0.5*link_2_height}" gazebo="${gazebo}">
+    <self_collision_geometries>
+      <xacro:collision_capsule xyz="0 0 0" radius="${link_2_radius+safety_distance}" length="${link_2_height+safety_distance}"/>
     </self_collision_geometries>
   </xacro:link_with_sc>
@@ -150,7 +159,7 @@
   </joint>
   <!--link3 to link2-->
-  <xacro:link_with_sc name="link3" link_height="${link_3_height}" link_radius="${link_3_radius}" pos_xyz="0 0 ${0.5*link_3_height}" pos_rpy="0 0 0" gazebo="${gazebo}">
-    <self_collision_geometries>
-      <xacro:collision_capsule xyz="0 0 0" radius="${link_1_radius+safety_distance}" length="${link_1_height+safety_distance}"/>
+  <xacro:link_with_sc name="link3" link_height="${link_3_height}" link_radius="${link_3_radius}" pos_xyz="0 0 ${0.5*link_3_height}" gazebo="${gazebo}">
+    <self_collision_geometries>
+      <xacro:collision_capsule xyz="0 0 0" radius="${link_3_radius+safety_distance}" length="${link_3_height+safety_distance}"/>
     </self_collision_geometries>
   </xacro:link_with_sc>
@@ -165,7 +174,7 @@
   </joint>
   <!--link4 to link3-->
-  <xacro:link_with_sc name="link4" link_height="${link_4_height}" link_radius="${link_4_radius}" pos_xyz="0 0 ${0.5*link_4_height}" pos_rpy="0 0 0" gazebo="${gazebo}">
-    <self_collision_geometries>
-      <xacro:collision_capsule xyz="0 0 0" radius="${link_1_radius+safety_distance}" length="${link_1_height+safety_distance}"/>
+  <xacro:link_with_sc name="link4" link_height="${link_4_height}" link_radius="${link_4_radius}" pos_xyz="0 0 ${0.5*link_4_height}" gazebo="${gazebo}">
+    <self_collision_geometries>
+      <xacro:collision_capsule xyz="0 0 0" radius="${link_4_radius+safety_distance}" length="${link_4_height+safety_distance}"/>
     </self_collision_geometries>
   </xacro:link_with_sc>
@@ -180,7 +189,7 @@
   </joint>
   <!--link5 to link4-->
-  <xacro:link_with_sc name="link5" link_height="${link_5_height}" link_radius="${link_5_radius}" pos_xyz="0 0 ${0.5*link_5_height}" pos_rpy="0 0 0" gazebo="${gazebo}">
-    <self_collision_geometries>
-      <xacro:collision_capsule xyz="0 0 0" radius="${link_1_radius+safety_distance}" length="${link_1_height+safety_distance}"/>
+  <xacro:link_with_sc name="link5" link_height="${link_5_height}" link_radius="${link_5_radius}" pos_xyz="0 0 ${0.5*link_5_height}" gazebo="${gazebo}">
+    <self_collision_geometries>
+      <xacro:collision_capsule xyz="0 0 0" radius="${link_5_radius+safety_distance}" length="${link_5_height+safety_distance}"/>
     </self_collision_geometries>
   </xacro:link_with_sc>
@@ -195,7 +204,7 @@
   </joint>
   <!--link6 to link5-->
-  <xacro:link_with_sc name="link6" link_height="${link_6_height}" link_radius="${link_6_radius}" pos_xyz="0 0 ${0.5*link_6_height}" pos_rpy="0 0 0" gazebo="${gazebo}">
-    <self_collision_geometries>
-      <xacro:collision_capsule xyz="0 0 0" radius="${link_1_radius+safety_distance}" length="${link_1_height+safety_distance}"/>
+  <xacro:link_with_sc name="link6" link_height="${link_6_height}" link_radius="${link_6_radius}" pos_xyz="0 0 ${0.5*link_6_height}" gazebo="${gazebo}">
+    <self_collision_geometries>
+      <xacro:collision_capsule xyz="0 0 0" radius="${link_6_radius+safety_distance}" length="${link_6_height+safety_distance}"/>
     </self_collision_geometries>
   </xacro:link_with_sc>
@@ -210,7 +219,7 @@
   </joint>
   <!--link7 to link6-->
-  <xacro:link_with_sc name="link7" link_height="${link_7_height}" link_radius="${link_7_radius}" pos_xyz="0 0 ${0.5*link_7_height}" pos_rpy="0 0 0" gazebo="${gazebo}">
-    <self_collision_geometries>
-      <xacro:collision_capsule xyz="0 0 0" radius="${link_1_radius+safety_distance}" length="${link_1_height+safety_distance}"/>
+  <xacro:link_with_sc name="link7" link_height="${link_7_height}" link_radius="${link_7_radius}" pos_xyz="0 0 ${0.5*link_7_height}" gazebo="${gazebo}">
+    <self_collision_geometries>
+      <xacro:collision_capsule xyz="0 0 0" radius="${link_7_radius+safety_distance}" length="${link_7_height+safety_distance}"/>
     </self_collision_geometries>
   </xacro:link_with_sc>
@@ -225,7 +234,7 @@
   </joint>
   <!--link8 to link7-->
-  <xacro:link_with_sc name="link8" link_height="${link_8_height}" link_radius="${link_8_radius}" pos_xyz="0 0 ${0.5*link_8_height}" pos_rpy="0 0 0" gazebo="${gazebo}">
-    <self_collision_geometries>
-      <xacro:collision_capsule xyz="0 0 0" radius="${link_1_radius+safety_distance}" length="${link_1_height+safety_distance}"/>
+  <xacro:link_with_sc name="link8" link_height="${link_8_height}" link_radius="${link_8_radius}" pos_xyz="0 0 ${0.5*link_8_height}" gazebo="${gazebo}">
+    <self_collision_geometries>
+      <xacro:collision_capsule xyz="0 0 0" radius="${link_8_radius+safety_distance}" length="${link_8_height+safety_distance}"/>
     </self_collision_geometries>
   </xacro:link_with_sc>
@@ -240,7 +249,7 @@
   </joint>
   <!--link9 to link8-->
-  <xacro:link_with_sc name="link9" link_height="${link_9_height}" link_radius="${link_9_radius}" pos_xyz="0 0 ${0.5*link_9_height}" pos_rpy="0 0 0" gazebo="${gazebo}">
-    <self_collision_geometries>
-      <xacro:collision_capsule xyz="0 0 0" radius="${link_1_radius+safety_distance}" length="${link_1_height+safety_distance}"/>
+  <xacro:link_with_sc name="link9" link_height="${link_9_height}" link_radius="${link_9_radius}" pos_xyz="0 0 ${0.5*link_9_height}" gazebo="${gazebo}">
+    <self_collision_geometries>
+      <xacro:collision_capsule xyz="0 0 0" radius="${link_9_radius+safety_distance}" length="${link_9_height+safety_distance}"/>
     </self_collision_geometries>
   </xacro:link_with_sc>
@@ -255,7 +264,7 @@
   </joint>
   <!--link10 to link9-->
-  <xacro:link_with_sc name="link10" link_height="${link_10_height}" link_radius="${link_10_radius}" pos_xyz="0 0 ${0.5*link_10_height}" pos_rpy="0 0 0" gazebo="${gazebo}">
-    <self_collision_geometries>
-      <xacro:collision_capsule xyz="0 0 0" radius="${link_1_radius+safety_distance}" length="${link_1_height+safety_distance}"/>
+  <xacro:link_with_sc name="link10" link_height="${link_10_height}" link_radius="${link_10_radius}" pos_xyz="0 0 ${0.5*link_10_height}" gazebo="${gazebo}">
+    <self_collision_geometries>
+      <xacro:collision_capsule xyz="0 0 0" radius="${link_10_radius+safety_distance}" length="${link_10_height+safety_distance}"/>
     </self_collision_geometries>
   </xacro:link_with_sc>
@@ -270,7 +279,7 @@
   </joint>
   <!--link11 to link10-->
-  <xacro:link_with_sc name="link11" link_height="${link_11_height}" link_radius="${link_11_radius}" pos_xyz="0 0 ${0.5*link_11_height}" pos_rpy="0 0 0" gazebo="${gazebo}">
-    <self_collision_geometries>
-      <xacro:collision_capsule xyz="0 0 0" radius="${link_1_radius+safety_distance}" length="${link_1_height+safety_distance}"/>
+  <xacro:link_with_sc name="link11" link_height="${link_11_height}" link_radius="${link_11_radius}" pos_xyz="0 0 ${0.5*link_11_height}" gazebo="${gazebo}">
+    <self_collision_geometries>
+      <xacro:collision_capsule xyz="0 0 0" radius="${link_11_radius+safety_distance}" length="${link_11_height+safety_distance}"/>
     </self_collision_geometries>
   </xacro:link_with_sc>
@@ -285,7 +294,7 @@
   </joint>
   <!--link12 to link11-->
-  <xacro:link_with_sc name="link12" link_height="${link_12_height}" link_radius="${link_12_radius}" pos_xyz="0 0 ${0.5*link_12_height}" pos_rpy="0 0 0" gazebo="${gazebo}">
-    <self_collision_geometries>
-      <xacro:collision_capsule xyz="0 0 0" radius="${link_1_radius+safety_distance}" length="${link_1_height+safety_distance}"/>
+  <xacro:link_with_sc name="link12" link_height="${link_12_height}" link_radius="${link_12_radius}" pos_xyz="0 0 ${0.5*link_12_height}" gazebo="${gazebo}">
+    <self_collision_geometries>
+      <xacro:collision_capsule xyz="0 0 0" radius="${link_12_radius+safety_distance}" length="${link_12_height+safety_distance}"/>
     </self_collision_geometries>
   </xacro:link_with_sc>
@@ -300,7 +309,7 @@
   </joint>
   <!--link13 to link12-->
-  <xacro:link_with_sc name="link13" link_height="${link_13_height}" link_radius="${link_13_radius}" pos_xyz="0 0 ${0.5*link_13_height}" pos_rpy="0 0 0" gazebo="${gazebo}">
-    <self_collision_geometries>
-      <xacro:collision_capsule xyz="0 0 0" radius="${link_1_radius+safety_distance}" length="${link_1_height+safety_distance}"/>
+  <xacro:link_with_sc name="link13" link_height="${link_13_height}" link_radius="${link_13_radius}" pos_xyz="0 0 ${0.5*link_13_height}" gazebo="${gazebo}">
+    <self_collision_geometries>
+      <xacro:collision_capsule xyz="0 0 0" radius="${link_13_radius+safety_distance}" length="${link_13_height+safety_distance}"/>
     </self_collision_geometries>
   </xacro:link_with_sc>

Commit message: revised limits and link radius

File: chin_description/urdf/chin_arm.urdf.xacro (robot description, xacro)
@@ -6,31 +6,31 @@
   <xacro:property name="safety_distance" value="0"/>
   <xacro:property name="link_base_height" value="0.204"/>
-  <xacro:property name="link_base_radius" value="0.2"/>
+  <xacro:property name="link_base_radius" value="0.095"/>
   <xacro:property name="link_1_height" value="0.081"/>
-  <xacro:property name="link_1_radius" value="0.02"/>
+  <xacro:property name="link_1_radius" value="0.066"/>
   <xacro:property name="link_2_height" value="0.082"/>
-  <xacro:property name="link_2_radius" value="0.02"/>
+  <xacro:property name="link_2_radius" value="0.066"/>
   <xacro:property name="link_3_height" value="0.07"/>
-  <xacro:property name="link_3_radius" value="0.02"/>
+  <xacro:property name="link_3_radius" value="0.066"/>
   <xacro:property name="link_4_height" value="0.398"/>
-  <xacro:property name="link_4_radius" value="0.02"/>
+  <xacro:property name="link_4_radius" value="0.055"/>
   <xacro:property name="link_5_height" value="0.065"/>
-  <xacro:property name="link_5_radius" value="0.02"/>
+  <xacro:property name="link_5_radius" value="0.055"/>
   <xacro:property name="link_6_height" value="0.063"/>
-  <xacro:property name="link_6_radius" value="0.02"/>
+  <xacro:property name="link_6_radius" value="0.055"/>
   <xacro:property name="link_7_height" value="0.36"/>
-  <xacro:property name="link_7_radius" value="0.02"/>
+  <xacro:property name="link_7_radius" value="0.045"/>
   <xacro:property name="link_8_height" value="0.083"/>
-  <xacro:property name="link_8_radius" value="0.02"/>
+  <xacro:property name="link_8_radius" value="0.045"/>
   <xacro:property name="link_9_height" value="0.087"/>
-  <xacro:property name="link_9_radius" value="0.02"/>
+  <xacro:property name="link_9_radius" value="0.045"/>
   <xacro:property name="link_10_height" value="0.083"/>
-  <xacro:property name="link_10_radius" value="0.02"/>
+  <xacro:property name="link_10_radius" value="0.045"/>
   <xacro:property name="link_11_height" value="0.087"/>
-  <xacro:property name="link_11_radius" value="0.02"/>
+  <xacro:property name="link_11_radius" value="0.045"/>
   <xacro:property name="link_12_height" value="0.083"/>
-  <xacro:property name="link_12_radius" value="0.02"/>
+  <xacro:property name="link_12_radius" value="0.045"/>
   <xacro:property name="link_13_height" value="0.077"/>
-  <xacro:property name="link_13_radius" value="0.02"/>
+  <xacro:property name="link_13_radius" value="0.045"/>
   <xacro:property name="with_mesh" value="false"/>
   <material name="white">
@@ -135,10 +135,10 @@
   </xacro:link_with_sc>
   <joint name="${arm_id}_joint1" type="revolute">
-    <safety_controller k_position="100.0" k_velocity="40.0" soft_lower_limit="-2.8973" soft_upper_limit="2.8973"/>
+    <safety_controller k_position="100.0" k_velocity="40.0" soft_lower_limit="${-pi}" soft_upper_limit="${pi}"/>
     <origin rpy="0 0 0" xyz="0 0 ${link_base_height}"/>
     <parent link="${arm_id}_link0"/>
     <child link="${arm_id}_link1"/>
-    <axis xyz="0 0 1" />
-    <limit lower="-2.8973" upper="2.8973" effort="0" velocity="0"/>
+    <axis xyz="0 0 1"/>
+    <limit lower="${-pi}" upper="${pi}" effort="0" velocity="0"/>
     <dynamics D="1" K="7000" damping="0.003" friction="0.0" mu_coulomb="0" mu_viscous="16"/>
   </joint>
@@ -150,10 +150,8 @@
   </xacro:link_with_sc>
   <joint name="${arm_id}_joint2" type="fixed">
-    <safety_controller k_position="100.0" k_velocity="40.0" soft_lower_limit="-2.8973" soft_upper_limit="2.8973"/>
     <origin rpy="${-0.5*pi} 0 0" xyz="0 0 ${link_1_height}"/>
     <parent link="${arm_id}_link1"/>
     <child link="${arm_id}_link2"/>
-    <axis xyz="0 0 1" />
-    <limit lower="-2.8973" upper="2.8973" effort="0" velocity="0"/>
+    <axis xyz="0 0 1"/>
     <dynamics D="1" K="7000" damping="0.003" friction="0.0" mu_coulomb="0" mu_viscous="16"/>
   </joint>
@@ -165,10 +163,10 @@
   </xacro:link_with_sc>
   <joint name="${arm_id}_joint3" type="revolute">
-    <safety_controller k_position="100.0" k_velocity="40.0" soft_lower_limit="-2.8973" soft_upper_limit="2.8973"/>
+    <safety_controller k_position="100.0" k_velocity="40.0" soft_lower_limit="${-pi}" soft_upper_limit="${pi}"/>
     <origin rpy="0 0 0" xyz="0 0 ${link_2_height}"/>
     <parent link="${arm_id}_link2"/>
     <child link="${arm_id}_link3"/>
-    <axis xyz="0 0 1" />
-    <limit lower="-2.8973" upper="2.8973" effort="0" velocity="0"/>
+    <axis xyz="0 0 1"/>
+    <limit lower="${-pi}" upper="${pi}" effort="0" velocity="0"/>
     <dynamics D="1" K="7000" damping="0.003" friction="0.0" mu_coulomb="0" mu_viscous="16"/>
   </joint>
@@ -180,10 +178,8 @@
   </xacro:link_with_sc>
   <joint name="${arm_id}_joint4" type="fixed">
-    <safety_controller k_position="100.0" k_velocity="40.0" soft_lower_limit="-2.8973" soft_upper_limit="2.8973"/>
     <origin rpy="${0.5*pi} 0 0" xyz="0 0 ${link_3_height}"/>
     <parent link="${arm_id}_link3"/>
     <child link="${arm_id}_link4"/>
-    <axis xyz="0 0 1" />
-    <limit lower="-2.8973" upper="2.8973" effort="0" velocity="0"/>
+    <axis xyz="0 0 1"/>
     <dynamics D="1" K="7000" damping="0.003" friction="0.0" mu_coulomb="0" mu_viscous="16"/>
   </joint>
@@ -195,10 +191,8 @@
   </xacro:link_with_sc>
   <joint name="${arm_id}_joint5" type="fixed">
-    <safety_controller k_position="100.0" k_velocity="40.0" soft_lower_limit="-2.8973" soft_upper_limit="2.8973"/>
     <origin rpy="${0.5*pi} 0 0" xyz="0 0 ${link_4_height}"/>
     <parent link="${arm_id}_link4"/>
     <child link="${arm_id}_link5"/>
-    <axis xyz="0 0 1" />
-    <limit lower="-2.8973" upper="2.8973" effort="0" velocity="0"/>
+    <axis xyz="0 0 1"/>
     <dynamics D="1" K="7000" damping="0.003" friction="0.0" mu_coulomb="0" mu_viscous="16"/>
   </joint>
@@ -210,10 +204,10 @@
   </xacro:link_with_sc>
   <joint name="${arm_id}_joint6" type="revolute">
-    <safety_controller k_position="100.0" k_velocity="40.0" soft_lower_limit="-2.8973" soft_upper_limit="2.8973"/>
+    <safety_controller k_position="100.0" k_velocity="40.0" soft_lower_limit="-2.7925" soft_upper_limit="2.7925"/>
     <origin rpy="0 0 0" xyz="0 0 ${link_5_height}"/>
     <parent link="${arm_id}_link5"/>
     <child link="${arm_id}_link6"/>
-    <axis xyz="0 0 1" />
-    <limit lower="-2.8973" upper="2.8973" effort="0" velocity="0"/>
+    <axis xyz="0 0 1"/>
+    <limit lower="-2.7925" upper="2.7925" effort="0" velocity="0"/>
     <dynamics D="1" K="7000" damping="0.003" friction="0.0" mu_coulomb="0" mu_viscous="16"/>
   </joint>
@@ -225,10 +219,8 @@
   </xacro:link_with_sc>
   <joint name="${arm_id}_joint7" type="fixed">
-    <safety_controller k_position="100.0" k_velocity="40.0" soft_lower_limit="-2.8973" soft_upper_limit="2.8973"/>
     <origin rpy="${-0.5*pi} 0 0" xyz="0 0 ${link_6_height}"/>
     <parent link="${arm_id}_link6"/>
     <child link="${arm_id}_link7"/>
-    <axis xyz="0 0 1" />
-    <limit lower="-2.8973" upper="2.8973" effort="0" velocity="0"/>
+    <axis xyz="0 0 1"/>
     <dynamics D="1" K="7000" damping="0.003" friction="0.0" mu_coulomb="0" mu_viscous="16"/>
   </joint>
@@ -240,10 +232,8 @@
   </xacro:link_with_sc>
   <joint name="${arm_id}_joint8" type="fixed">
-    <safety_controller k_position="100.0" k_velocity="40.0" soft_lower_limit="-2.8973" soft_upper_limit="2.8973"/>
     <origin rpy="${-0.5*pi} 0 0" xyz="0 0 ${link_7_height}"/>
     <parent link="${arm_id}_link7"/>
     <child link="${arm_id}_link8"/>
-    <axis xyz="0 0 1" />
-    <limit lower="-2.8973" upper="2.8973" effort="0" velocity="0"/>
+    <axis xyz="0 0 1"/>
     <dynamics D="1" K="7000" damping="0.003" friction="0.0" mu_coulomb="0" mu_viscous="16"/>
   </joint>
@@ -255,10 +245,10 @@
   </xacro:link_with_sc>
   <joint name="${arm_id}_joint9" type="revolute">
-    <safety_controller k_position="100.0" k_velocity="40.0" soft_lower_limit="-2.8973" soft_upper_limit="2.8973"/>
+    <safety_controller k_position="100.0" k_velocity="40.0" soft_lower_limit="${-pi}" soft_upper_limit="${pi}"/>
     <origin rpy="0 0 0" xyz="0 0 ${link_8_height}"/>
     <parent link="${arm_id}_link8"/>
     <child link="${arm_id}_link9"/>
-    <axis xyz="0 0 1" />
-    <limit lower="-2.8973" upper="2.8973" effort="0" velocity="0"/>
+    <axis xyz="0 0 1"/>
+    <limit lower="${-pi}" upper="${pi}" effort="0" velocity="0"/>
     <dynamics D="1" K="7000" damping="0.003" friction="0.0" mu_coulomb="0" mu_viscous="16"/>
   </joint>
@@ -270,10 +260,8 @@
   </xacro:link_with_sc>
   <joint name="${arm_id}_joint10" type="fixed">
-    <safety_controller k_position="100.0" k_velocity="40.0" soft_lower_limit="-2.8973" soft_upper_limit="2.8973"/>
     <origin rpy="${0.5*pi} 0 0" xyz="0 0 ${link_9_height}"/>
     <parent link="${arm_id}_link9"/>
     <child link="${arm_id}_link10"/>
-    <axis xyz="0 0 1" />
-    <limit lower="-2.8973" upper="2.8973" effort="0" velocity="0"/>
+    <axis xyz="0 0 1"/>
     <dynamics D="1" K="7000" damping="0.003" friction="0.0" mu_coulomb="0" mu_viscous="16"/>
   </joint>
@@ -285,10 +273,10 @@
   </xacro:link_with_sc>
   <joint name="${arm_id}_joint11" type="revolute">
-    <safety_controller k_position="100.0" k_velocity="40.0" soft_lower_limit="-2.8973" soft_upper_limit="2.8973"/>
+    <safety_controller k_position="100.0" k_velocity="40.0" soft_lower_limit="${-pi}" soft_upper_limit="${pi}"/>
     <origin rpy="0 0 0" xyz="0 0 ${link_10_height}"/>
     <parent link="${arm_id}_link10"/>
     <child link="${arm_id}_link11"/>
-    <axis xyz="0 0 1" />
-    <limit lower="-2.8973" upper="2.8973" effort="0" velocity="0"/>
+    <axis xyz="0 0 1"/>
+    <limit lower="${-pi}" upper="${pi}" effort="0" velocity="0"/>
     <dynamics D="1" K="7000" damping="0.003" friction="0.0" mu_coulomb="0" mu_viscous="16"/>
   </joint>
@@ -300,10 +288,8 @@
   </xacro:link_with_sc>
   <joint name="${arm_id}_joint12" type="fixed">
-    <safety_controller k_position="100.0" k_velocity="40.0" soft_lower_limit="-2.8973" soft_upper_limit="2.8973"/>
     <origin rpy="${-0.5*pi} 0 0" xyz="0 0 ${link_11_height}"/>
     <parent link="${arm_id}_link11"/>
     <child link="${arm_id}_link12"/>
-    <axis xyz="0 0 1" />
-    <limit lower="-2.8973" upper="2.8973" effort="0" velocity="0"/>
+    <axis xyz="0 0 1"/>
     <dynamics D="1" K="7000" damping="0.003" friction="0.0" mu_coulomb="0" mu_viscous="16"/>
   </joint>
@@ -315,10 +301,10 @@
   </xacro:link_with_sc>
   <joint name="${arm_id}_joint13" type="revolute">
-    <safety_controller k_position="100.0" k_velocity="40.0" soft_lower_limit="-2.8973" soft_upper_limit="2.8973"/>
+    <safety_controller k_position="100.0" k_velocity="40.0" soft_lower_limit="${-pi}" soft_upper_limit="${pi}"/>
     <origin rpy="0 0 0" xyz="0 0 ${link_12_height}"/>
     <parent link="${arm_id}_link12"/>
     <child link="${arm_id}_link13"/>
-    <axis xyz="0 0 1" />
-    <limit lower="-2.8973" upper="2.8973" effort="0" velocity="0"/>
+    <axis xyz="0 0 1"/>
+    <limit lower="${-pi}" upper="${pi}" effort="0" velocity="0"/>
     <dynamics D="1" K="7000" damping="0.003" friction="0.0" mu_coulomb="0" mu_viscous="16"/>
   </joint>

Commit message: align TCP orientation

File: chin_description/urdf/chin_arm.urdf.xacro (robot description, xacro)
@@ -312,5 +312,5 @@
   <link name="${arm_id}_link14"/>
   <joint name="${arm_id}_joint14" type="fixed">
-    <origin rpy="0 0 0" xyz="0 0 ${link_13_height}"/>
+    <origin rpy="0 0 ${-pi}" xyz="0 0 ${link_13_height}"/>
     <parent link="${arm_id}_link13"/>
     <child link="${arm_id}_link14"/>
