Commit message: valid mesh urdf

File: chin_description/urdf/chin_arm.urdf.xacro (robot description, xacro)
@@ -5,5 +5,5 @@
   <xacro:property name="gazebo" value="false"/>
   <xacro:property name="safety_distance" value="0"/>
-  <xacro:property name="link_base_height" value="0.204"/>
+  <xacro:property name="link_base_height" value="0.2038"/>
   <xacro:property name="link_base_radius" value="0.095"/>
   <xacro:property name="link_1_height" value="0.081"/>
@@ -135,7 +135,5 @@
   <!--link1 to link0-->
   <xacro:link_with_sc name="link_1" link_height="${link_1_height}" link_radius="${link_1_radius}" pos_xyz="0 0 0" gazebo="${gazebo}">
-    <self_collision_geometries>
-      <xacro:collision_capsule xyz="0 0 ${0.5*link_1_height}" radius="${link_1_radius+safety_distance}" length="${link_1_height+safety_distance}"/>
-    </self_collision_geometries>
+    <self_collision_geometries/>
   </xacro:link_with_sc>
   <joint name="${arm_id}_joint_1" type="revolute">
@@ -150,7 +148,5 @@
   <!--link2 to link1-->
   <xacro:link_with_sc name="link_2" link_height="${link_2_height}" link_radius="${link_2_radius}" pos_xyz="0 0 0" gazebo="${gazebo}">
-    <self_collision_geometries>
-      <xacro:collision_capsule xyz="0 0 ${0.5*link_2_height}" radius="${link_2_radius+safety_distance}" length="${link_2_height+safety_distance}"/>
-    </self_collision_geometries>
+    <self_collision_geometries/>
   </xacro:link_with_sc>
   <joint name="${arm_id}_joint_2" type="revolute">
@@ -165,26 +161,22 @@
   <!--link3 to link2-->
   <xacro:link_with_sc name="link_3" link_height="${link_3_height}" link_radius="${link_3_radius}" pos_xyz="0 0 0" gazebo="${gazebo}">
-    <self_collision_geometries>
-      <xacro:collision_capsule xyz="0 0 ${0.5*link_3_height}" radius="${link_3_radius+safety_distance}" length="${link_2_height+safety_distance}"/>
-    </self_collision_geometries>
+    <self_collision_geometries/>
   </xacro:link_with_sc>
   <joint name="${arm_id}_joint_3" type="revolute">
-    <safety_controller k_position="100.0" k_velocity="40.0" soft_lower_limit="${-pi}" soft_upper_limit="${pi}"/>
-    <origin rpy="${pi} 0 0" xyz="0 ${-link_4_height} 0"/>
+    <safety_controller k_position="100.0" k_velocity="40.0" soft_lower_limit="-2.7925" soft_upper_limit="2.7925"/>
+    <origin rpy="${pi} 0 0" xyz="0 ${-link_4_height} 0.0045"/>
     <parent link="${arm_id}_link_2"/>
     <child link="${arm_id}_link_3"/>
     <axis xyz="0 0 1"/>
-    <limit lower="${-pi}" upper="${pi}" effort="0" velocity="0"/>
+    <limit lower="-2.7925" upper="2.7925" effort="0" velocity="0"/>
     <dynamics D="1" K="7000" damping="0.003" friction="0.0" mu_coulomb="0" mu_viscous="16"/>
   </joint>
   <!--link4 to link3-->
   <xacro:link_with_sc name="link_4" link_height="${link_4_height}" link_radius="${link_4_radius}" pos_xyz="0 0 0" gazebo="${gazebo}">
-    <self_collision_geometries>
-      <xacro:collision_capsule xyz="0 0 ${0.5*link_4_height}" radius="${link_4_radius+safety_distance}" length="${link_4_height+safety_distance}"/>
-    </self_collision_geometries>
+    <self_collision_geometries/>
   </xacro:link_with_sc>
   <joint name="${arm_id}_joint_4" type="revolute">
     <safety_controller k_position="100.0" k_velocity="40.0" soft_lower_limit="${-pi}" soft_upper_limit="${pi}"/>
-    <origin rpy="${pi} 0 0" xyz="0 ${link_7_height} ${link_6_height-link_8_height}"/>
+    <origin rpy="${pi} 0 0" xyz="0 ${link_7_height} -0.0202"/>
     <parent link="${arm_id}_link_3"/>
     <child link="${arm_id}_link_4"/>
@@ -195,7 +187,5 @@
   <!--link5 to link4-->
   <xacro:link_with_sc name="link_5" link_height="${link_5_height}" link_radius="${link_5_radius}" pos_xyz="0 0 0" gazebo="${gazebo}">
-    <self_collision_geometries>
-      <xacro:collision_capsule xyz="0 0 ${0.5*link_5_height}" radius="${link_5_radius+safety_distance}" length="${link_5_height+safety_distance}"/>
-    </self_collision_geometries>
+    <self_collision_geometries/>
   </xacro:link_with_sc>
   <joint name="${arm_id}_joint_5" type="revolute">
@@ -210,7 +200,5 @@
   <!--link6 to link5-->
   <xacro:link_with_sc name="link_6" link_height="${link_6_height}" link_radius="${link_6_radius}" pos_xyz="0 0 0" gazebo="${gazebo}">
-    <self_collision_geometries>
-      <xacro:collision_capsule xyz="0 0 ${0.5*link_6_height}" radius="${link_6_radius+safety_distance}" length="${link_6_height+safety_distance}"/>
-    </self_collision_geometries>
+    <self_collision_geometries/>
   </xacro:link_with_sc>
   <joint name="${arm_id}_joint_6" type="revolute">

Commit message: mesh urdf valid version

File: chin_description/urdf/chin_arm.urdf.xacro (robot description, xacro)
@@ -4,5 +4,4 @@
   <!--is the robot being simulated in gazebo?-->
   <xacro:property name="gazebo" value="false"/>
-  <xacro:property name="safety_distance" value="0"/>
   <xacro:property name="link_base_height" value="0.2038"/>
   <xacro:property name="link_base_radius" value="0.095"/>
@@ -44,45 +43,4 @@
     <color rgba="0.51 0.54 0.59 1"/>
   </material>
-  <!-- =========================================================== -->
-  <!-- add a <collision> tag with a capsule, made from a cylinder  -->
-  <!-- with two spheres at its caps. The capsule will always be    -->
-  <!-- aligned with the axis of 'direction' you pass along.        -->
-  <!--                                                             -->
-  <!-- radius: Radii of both the cylinder and both spheres [m]     -->
-  <!-- length: Length of the cylinder/distance between the centers -->
-  <!--         of the spheres. NOT overall length of capsule!      -->
-  <!-- xyz:    Position of the center of the capsule/cylinder      -->
-  <!-- direction: One of { x, y, z, -x, -y, -z }                   -->
-  <!-- =========================================================== -->
-  <xacro:macro name="collision_capsule" params="radius length xyz:='0 0 0' direction:='z'">
-    <xacro:property name="r" value="${0.5*pi if 'y' in direction else 0}"/>
-    <xacro:property name="p" value="${0.5*pi if 'x' in direction else 0}"/>
-    <xacro:property name="y" value="0"/>
-    <xacro:property name="x" value="${xyz.split(' ')[0]}"/>
-    <xacro:property name="y" value="${xyz.split(' ')[1]}"/>
-    <xacro:property name="z" value="${xyz.split(' ')[2]}"/>
-    <!--sphere center offsets from center of cylinder-->
-    <xacro:property name="sx" value="${0.5*length if 'x' in direction else 0}"/>
-    <xacro:property name="sy" value="${0.5*length if 'y' in direction else 0}"/>
-    <xacro:property name="sz" value="${0.5*length if 'z' in direction else 0}"/>
-    <collision>
-      <origin xyz="${x} ${y} ${z}" rpy="${r} ${p} ${y}"/>
-      <geometry>
-        <cylinder radius="${radius}" length="${length}"/>
-      </geometry>
-    </collision>
-    <collision>
-      <origin xyz="${x+sx} ${y+sy} ${z+sz}"/>
-      <geometry>
-        <sphere radius="${radius}"/>
-      </geometry>
-    </collision>
-    <collision>
-      <origin xyz="${x-sx} ${y-sy} ${z-sz}"/>
-      <geometry>
-        <sphere radius="${radius}"/>
-      </geometry>
-    </collision>
-  </xacro:macro>
   <xacro:macro name="link_with_sc"  params="name link_height link_radius pos_xyz:='0 0 0' pos_rpy:='0 0 0' visual_color:='white' prefix=${arm_id} rpy:='0 0 0' **self_collision_geometries gazebo:=false">
     <!--sub-link defining detailed meshes for collision with environment-->
@@ -99,5 +57,7 @@
           </xacro:unless>
         </geometry>
-        <material name="${visual_color}"/>
+        <xacro:unless value="${mesh == 'yes'}">
+          <material name="${visual_color}"/>
+        </xacro:unless>
       </visual>
       <collision>
@@ -116,19 +76,7 @@
       </xacro:if>
     </link>
-    <!--sub-link defining coarse geometries of real robot's internal self-collision-->
-    <link name="${prefix}_${name}_sc">
-      <xacro:unless value="${gazebo}">
-        <xacro:insert_block name="self_collision_geometries"/>
-      </xacro:unless>
-    </link>
-    <!--fixed joint between both sub-links-->
-    <joint name="${prefix}_${name}_sc_joint" type="fixed">
-      <origin rpy="${rpy}"/>
-      <parent link="${prefix}_${name}"/>
-      <child link="${prefix}_${name}_sc"/>
-    </joint>
   </xacro:macro>
   <!--fixed link0-->
-  <xacro:link_with_sc name="link_0" link_height="${link_base_height}" link_radius="${link_base_radius}" visual_color="black" gazebo="${gazebo}">
+  <xacro:link_with_sc name="link_0" link_height="${link_base_height}" link_radius="${link_base_radius}" gazebo="${gazebo}">
     <self_collision_geometries/>
   </xacro:link_with_sc>
@@ -138,10 +86,10 @@
   </xacro:link_with_sc>
   <joint name="${arm_id}_joint_1" type="revolute">
-    <safety_controller k_position="100.0" k_velocity="40.0" soft_lower_limit="${-pi}" soft_upper_limit="${pi}"/>
+    <safety_controller k_position="100.0" k_velocity="40.0" soft_lower_limit="-${pi}" soft_upper_limit="${pi}"/>
     <origin rpy="0 0 0" xyz="0 0 ${link_base_height}"/>
     <parent link="${arm_id}_link_0"/>
     <child link="${arm_id}_link_1"/>
     <axis xyz="0 0 1"/>
-    <limit lower="${-pi}" upper="${pi}" effort="0" velocity="0"/>
+    <limit lower="-${pi}" upper="${pi}" effort="0" velocity="0"/>
     <dynamics D="1" K="7000" damping="0.003" friction="0.0" mu_coulomb="0" mu_viscous="16"/>
   </joint>
@@ -151,10 +99,10 @@
   </xacro:link_with_sc>
   <joint name="${arm_id}_joint_2" type="revolute">
-    <safety_controller k_position="100.0" k_velocity="40.0" soft_lower_limit="${-pi}" soft_upper_limit="${pi}"/>
+    <safety_controller k_position="100.0" k_velocity="40.0" soft_lower_limit="-${pi}" soft_upper_limit="${pi}"/>
     <origin rpy="${-0.5*pi} 0 0" xyz="0 ${link_2_height} ${link_1_height}"/>
     <parent link="${arm_id}_link_1"/>
     <child link="${arm_id}_link_2"/>
     <axis xyz="0 0 1"/>
-    <limit lower="${-pi}" upper="${pi}" effort="0" velocity="0"/>
+    <limit lower="-${pi}" upper="${pi}" effort="0" velocity="0"/>
     <dynamics D="1" K="7000" damping="0.003" friction="0.0" mu_coulomb="0" mu_viscous="16"/>
   </joint>
@@ -165,5 +113,5 @@
   <joint name="${arm_id}_joint_3" type="revolute">
     <safety_controller k_position="100.0" k_velocity="40.0" soft_lower_limit="-2.7925" soft_upper_limit="2.7925"/>
-    <origin rpy="${pi} 0 0" xyz="0 ${-link_4_height} 0.0045"/>
+    <origin rpy="${pi} 0 0" xyz="0 -${link_4_height} 0"/>
     <parent link="${arm_id}_link_2"/>
     <child link="${arm_id}_link_3"/>
@@ -177,10 +125,10 @@
   </xacro:link_with_sc>
   <joint name="${arm_id}_joint_4" type="revolute">
-    <safety_controller k_position="100.0" k_velocity="40.0" soft_lower_limit="${-pi}" soft_upper_limit="${pi}"/>
-    <origin rpy="${pi} 0 0" xyz="0 ${link_7_height} -0.0202"/>
+    <safety_controller k_position="100.0" k_velocity="40.0" soft_lower_limit="-${pi}" soft_upper_limit="${pi}"/>
+    <origin rpy="${pi} 0 0" xyz="0 ${link_7_height} -${link_8_height-link_6_height}"/>
     <parent link="${arm_id}_link_3"/>
     <child link="${arm_id}_link_4"/>
     <axis xyz="0 0 1"/>
-    <limit lower="${-pi}" upper="${pi}" effort="0" velocity="0"/>
+    <limit lower="-${pi}" upper="${pi}" effort="0" velocity="0"/>
     <dynamics D="1" K="7000" damping="0.003" friction="0.0" mu_coulomb="0" mu_viscous="16"/>
   </joint>
@@ -191,9 +139,9 @@
   <joint name="${arm_id}_joint_5" type="revolute">
     <safety_controller k_position="100.0" k_velocity="40.0" soft_lower_limit="${-pi}" soft_upper_limit="${pi}"/>
-    <origin rpy="${0.5*pi} 0 0" xyz="0 ${-link_10_height} ${link_11_height}"/>
+    <origin rpy="${0.5*pi} 0 0" xyz="0 -${link_10_height} ${link_11_height}"/>
     <parent link="${arm_id}_link_4"/>
     <child link="${arm_id}_link_5"/>
     <axis xyz="0 0 1"/>
-    <limit lower="${-pi}" upper="${pi}" effort="0" velocity="0"/>
+    <limit lower="-${pi}" upper="${pi}" effort="0" velocity="0"/>
     <dynamics D="1" K="7000" damping="0.003" friction="0.0" mu_coulomb="0" mu_viscous="16"/>
   </joint>
@@ -203,10 +151,10 @@
   </xacro:link_with_sc>
   <joint name="${arm_id}_joint_6" type="revolute">
-    <safety_controller k_position="100.0" k_velocity="40.0" soft_lower_limit="${-pi}" soft_upper_limit="${pi}"/>
+    <safety_controller k_position="100.0" k_velocity="40.0" soft_lower_limit="-${pi}" soft_upper_limit="${pi}"/>
     <origin rpy="${-0.5*pi} 0 0" xyz="0 ${link_12_height} ${link_11_height}"/>
     <parent link="${arm_id}_link_5"/>
     <child link="${arm_id}_link_6"/>
     <axis xyz="0 0 1"/>
-    <limit lower="${-pi}" upper="${pi}" effort="0" velocity="0"/>
+    <limit lower="-${pi}" upper="${pi}" effort="0" velocity="0"/>
     <dynamics D="1" K="7000" damping="0.003" friction="0.0" mu_coulomb="0" mu_viscous="16"/>
   </joint>
@@ -214,5 +162,5 @@
   <link name="${arm_id}_link_7"/>
   <joint name="${arm_id}_joint_7" type="fixed">
-    <origin rpy="0 0 ${-pi}" xyz="0 0 ${link_13_height}"/>
+    <origin rpy="0 0 -${pi}" xyz="0 0 ${link_13_height}"/>
     <parent link="${arm_id}_link_6"/>
     <child link="${arm_id}_link_7"/>

File: chin_description/urdf/chin_arm_frame.urdf.xacro (robot description, xacro)
@@ -99,5 +99,7 @@
           </xacro:unless>
         </geometry>
-        <material name="${visual_color}"/>
+        <xacro:unless value="${mesh == 'yes'}">
+          <material name="${visual_color}"/>
+        </xacro:unless>
       </visual>
       <collision>
@@ -134,5 +136,5 @@
   </xacro:link_with_sc>
   <!--link1 to link0-->
-  <xacro:link_with_sc name="link1" link_height="${link_1_height}" link_radius="${link_1_radius}" pos_xyz="0 0 ${0.5*link_1_height}" gazebo="${gazebo}">
+  <xacro:link_with_sc name="link1" link_height="${link_1_height}" link_radius="${link_1_radius}" pos_xyz="0 0 ${0.5*link_1_height}" visual_color="silver" gazebo="${gazebo}">
     <self_collision_geometries>
       <xacro:collision_capsule xyz="0 0 ${0.5*link_1_height}" radius="${link_1_radius+safety_distance}" length="${link_1_height+safety_distance}"/>
@@ -140,10 +142,10 @@
   </xacro:link_with_sc>
   <joint name="${arm_id}_joint1" type="revolute">
-    <safety_controller k_position="100.0" k_velocity="40.0" soft_lower_limit="${-pi}" soft_upper_limit="${pi}"/>
+    <safety_controller k_position="100.0" k_velocity="40.0" soft_lower_limit="-${pi}" soft_upper_limit="${pi}"/>
     <origin rpy="0 0 0" xyz="0 0 ${link_base_height}"/>
     <parent link="${arm_id}_link0"/>
     <child link="${arm_id}_link1"/>
     <axis xyz="0 0 1"/>
-    <limit lower="${-pi}" upper="${pi}" effort="0" velocity="0"/>
+    <limit lower="-${pi}" upper="${pi}" effort="0" velocity="0"/>
     <dynamics D="1" K="7000" damping="0.003" friction="0.0" mu_coulomb="0" mu_viscous="16"/>
   </joint>
@@ -155,5 +157,5 @@
   </xacro:link_with_sc>
   <joint name="${arm_id}_joint2" type="fixed">
-    <origin rpy="${-0.5*pi} 0 0" xyz="0 0 ${link_1_height}"/>
+    <origin rpy="-${0.5*pi} 0 0" xyz="0 0 ${link_1_height}"/>
     <parent link="${arm_id}_link1"/>
     <child link="${arm_id}_link2"/>
@@ -162,5 +164,5 @@
   </joint>
   <!--link3 to link2-->
-  <xacro:link_with_sc name="link3" link_height="${link_3_height}" link_radius="${link_3_radius}" pos_xyz="0 0 ${0.5*link_3_height}" gazebo="${gazebo}">
+  <xacro:link_with_sc name="link3" link_height="${link_3_height}" link_radius="${link_3_radius}" pos_xyz="0 0 ${0.5*link_3_height}" visual_color="silver" gazebo="${gazebo}">
     <self_collision_geometries>
       <xacro:collision_capsule xyz="0 0 ${0.5*link_3_height}" radius="${link_3_radius+safety_distance}" length="${link_3_height+safety_distance}"/>
@@ -168,10 +170,10 @@
   </xacro:link_with_sc>
   <joint name="${arm_id}_joint3" type="revolute">
-    <safety_controller k_position="100.0" k_velocity="40.0" soft_lower_limit="${-pi}" soft_upper_limit="${pi}"/>
+    <safety_controller k_position="100.0" k_velocity="40.0" soft_lower_limit="-${pi}" soft_upper_limit="${pi}"/>
     <origin rpy="0 0 0" xyz="0 0 ${link_2_height}"/>
     <parent link="${arm_id}_link2"/>
     <child link="${arm_id}_link3"/>
     <axis xyz="0 0 1"/>
-    <limit lower="${-pi}" upper="${pi}" effort="0" velocity="0"/>
+    <limit lower="-${pi}" upper="${pi}" effort="0" velocity="0"/>
     <dynamics D="1" K="7000" damping="0.003" friction="0.0" mu_coulomb="0" mu_viscous="16"/>
   </joint>
@@ -203,5 +205,5 @@
   </joint>
   <!--link6 to link5-->
-  <xacro:link_with_sc name="link6" link_height="${link_6_height}" link_radius="${link_6_radius}" pos_xyz="0 0 ${0.5*link_6_height}" gazebo="${gazebo}">
+  <xacro:link_with_sc name="link6" link_height="${link_6_height}" link_radius="${link_6_radius}" pos_xyz="0 0 ${0.5*link_6_height}" visual_color="silver" gazebo="${gazebo}">
     <self_collision_geometries>
       <xacro:collision_capsule xyz="0 0 ${0.5*link_6_height}" radius="${link_6_radius+safety_distance}" length="${link_6_height+safety_distance}"/>
@@ -224,5 +226,5 @@
   </xacro:link_with_sc>
   <joint name="${arm_id}_joint7" type="fixed">
-    <origin rpy="${-0.5*pi} 0 0" xyz="0 0 ${link_6_height}"/>
+    <origin rpy="-${0.5*pi} 0 0" xyz="0 0 ${link_6_height}"/>
     <parent link="${arm_id}_link6"/>
     <child link="${arm_id}_link7"/>
@@ -237,5 +239,5 @@
   </xacro:link_with_sc>
   <joint name="${arm_id}_joint8" type="fixed">
-    <origin rpy="${-0.5*pi} 0 0" xyz="0 0 ${link_7_height}"/>
+    <origin rpy="-${0.5*pi} 0 0" xyz="0 0 ${link_7_height}"/>
     <parent link="${arm_id}_link7"/>
     <child link="${arm_id}_link8"/>
@@ -244,5 +246,5 @@
   </joint>
   <!--link9 to link8-->
-  <xacro:link_with_sc name="link9" link_height="${link_9_height}" link_radius="${link_9_radius}" pos_xyz="0 0 ${0.5*link_9_height}" gazebo="${gazebo}">
+  <xacro:link_with_sc name="link9" link_height="${link_9_height}" link_radius="${link_9_radius}" pos_xyz="0 0 ${0.5*link_9_height}" visual_color="silver" gazebo="${gazebo}">
     <self_collision_geometries>
       <xacro:collision_capsule xyz="0 0 ${0.5*link_9_height}" radius="${link_9_radius+safety_distance}" length="${link_9_height+safety_distance}"/>
@@ -250,10 +252,10 @@
   </xacro:link_with_sc>
   <joint name="${arm_id}_joint9" type="revolute">
-    <safety_controller k_position="100.0" k_velocity="40.0" soft_lower_limit="${-pi}" soft_upper_limit="${pi}"/>
+    <safety_controller k_position="100.0" k_velocity="40.0" soft_lower_limit="-${pi}" soft_upper_limit="${pi}"/>
     <origin rpy="0 0 0" xyz="0 0 ${link_8_height}"/>
     <parent link="${arm_id}_link8"/>
     <child link="${arm_id}_link9"/>
     <axis xyz="0 0 1"/>
-    <limit lower="${-pi}" upper="${pi}" effort="0" velocity="0"/>
+    <limit lower="-${pi}" upper="${pi}" effort="0" velocity="0"/>
     <dynamics D="1" K="7000" damping="0.003" friction="0.0" mu_coulomb="0" mu_viscous="16"/>
   </joint>
@@ -272,5 +274,5 @@
   </joint>
   <!--link11 to link10-->
-  <xacro:link_with_sc name="link11" link_height="${link_11_height}" link_radius="${link_11_radius}" pos_xyz="0 0 ${0.5*link_11_height}" gazebo="${gazebo}">
+  <xacro:link_with_sc name="link11" link_height="${link_11_height}" link_radius="${link_11_radius}" pos_xyz="0 0 ${0.5*link_11_height}" visual_color="silver" gazebo="${gazebo}">
     <self_collision_geometries>
       <xacro:collision_capsule xyz="0 0 ${0.5*link_11_height}" radius="${link_11_radius+safety_distance}" length="${link_11_height+safety_distance}"/>
@@ -278,10 +280,10 @@
   </xacro:link_with_sc>
   <joint name="${arm_id}_joint11" type="revolute">
-    <safety_controller k_position="100.0" k_velocity="40.0" soft_lower_limit="${-pi}" soft_upper_limit="${pi}"/>
+    <safety_controller k_position="100.0" k_velocity="40.0" soft_lower_limit="-${pi}" soft_upper_limit="${pi}"/>
     <origin rpy="0 0 0" xyz="0 0 ${link_10_height}"/>
     <parent link="${arm_id}_link10"/>
     <child link="${arm_id}_link11"/>
     <axis xyz="0 0 1"/>
-    <limit lower="${-pi}" upper="${pi}" effort="0" velocity="0"/>
+    <limit lower="-${pi}" upper="${pi}" effort="0" velocity="0"/>
     <dynamics D="1" K="7000" damping="0.003" friction="0.0" mu_coulomb="0" mu_viscous="16"/>
   </joint>
@@ -293,5 +295,5 @@
   </xacro:link_with_sc>
   <joint name="${arm_id}_joint12" type="fixed">
-    <origin rpy="${-0.5*pi} 0 0" xyz="0 0 ${link_11_height}"/>
+    <origin rpy="-${0.5*pi} 0 0" xyz="0 0 ${link_11_height}"/>
     <parent link="${arm_id}_link11"/>
     <child link="${arm_id}_link12"/>
@@ -300,5 +302,5 @@
   </joint>
   <!--link13 to link12-->
-  <xacro:link_with_sc name="link13" link_height="${link_13_height}" link_radius="${link_13_radius}" pos_xyz="0 0 ${0.5*link_13_height}" gazebo="${gazebo}" visual_color="silver">
+  <xacro:link_with_sc name="link13" link_height="${link_13_height}" link_radius="${link_13_radius}" pos_xyz="0 0 ${0.5*link_13_height}" visual_color="silver" gazebo="${gazebo}">
     <self_collision_geometries>
       <xacro:collision_capsule xyz="0 0 ${0.5*link_13_height}" radius="${link_13_radius+safety_distance}" length="${link_13_height+safety_distance}"/>
@@ -306,10 +308,10 @@
   </xacro:link_with_sc>
   <joint name="${arm_id}_joint13" type="revolute">
-    <safety_controller k_position="100.0" k_velocity="40.0" soft_lower_limit="${-pi}" soft_upper_limit="${pi}"/>
+    <safety_controller k_position="100.0" k_velocity="40.0" soft_lower_limit="-${pi}" soft_upper_limit="${pi}"/>
     <origin rpy="0 0 0" xyz="0 0 ${link_12_height}"/>
     <parent link="${arm_id}_link12"/>
     <child link="${arm_id}_link13"/>
     <axis xyz="0 0 1"/>
-    <limit lower="${-pi}" upper="${pi}" effort="0" velocity="0"/>
+    <limit lower="-${pi}" upper="${pi}" effort="0" velocity="0"/>
     <dynamics D="1" K="7000" damping="0.003" friction="0.0" mu_coulomb="0" mu_viscous="16"/>
   </joint>
@@ -317,5 +319,5 @@
   <link name="${arm_id}_link14"/>
   <joint name="${arm_id}_joint14" type="fixed">
-    <origin rpy="0 0 ${-pi}" xyz="0 0 ${link_13_height}"/>
+    <origin rpy="0 0 -${pi}" xyz="0 0 ${link_13_height}"/>
     <parent link="${arm_id}_link13"/>
     <child link="${arm_id}_link14"/>
