Commit message: rename for further model extension

File: chin_crb7_description/urdf/chin_crb7.urdf.xacro (robot description, xacro)
@@ -2,4 +2,7 @@
 <robot name="chin_arm" xmlns:xacro="http://ros.org/wiki/xacro">
   <xacro:property name="arm_id" value="chin"/>
+  <xacro:property name="arm_model" value="crb7"/>
+  <xacro:property name="description_pkg" value="${arm_id}_${arm_model}_description"/>
+  <xacro:property name="mesh" value="yes"/>
   <!--is the robot being simulated in gazebo?-->
   <xacro:property name="gazebo" value="false"/>
@@ -32,6 +35,4 @@
   <xacro:property name="link_13_height" value="0.077"/>
   <xacro:property name="link_13_radius" value="0.045"/>
-  <xacro:property name="mesh" value="yes"/>
-  <xacro:property name="description_pkg" value="${arm_id}_description"/>
   <material name="white">
     <color rgba="1 1 1 1"/>

File: chin_crb7_moveit_config/config/gazebo_chin_arm.urdf (robot description, URDF)
Before this commit: robot chin_arm, 8 links, 7 joints
Links:
- link chin_link_0: geometry collision mesh filename=package://chin_crb7_description/meshes/collision/link_0.stl; visual mesh filename=package://chin_crb7_description/meshes/visual/link_0.dae
- link chin_link_1: geometry collision mesh filename=package://chin_crb7_description/meshes/collision/link_1.stl; visual mesh filename=package://chin_crb7_description/meshes/visual/link_1.dae
- link chin_link_2: geometry collision mesh filename=package://chin_crb7_description/meshes/collision/link_2.stl; visual mesh filename=package://chin_crb7_description/meshes/visual/link_2.dae
- link chin_link_3: geometry collision mesh filename=package://chin_crb7_description/meshes/collision/link_3.stl; visual mesh filename=package://chin_crb7_description/meshes/visual/link_3.dae
- link chin_link_4: geometry collision mesh filename=package://chin_crb7_description/meshes/collision/link_4.stl; visual mesh filename=package://chin_crb7_description/meshes/visual/link_4.dae
- link chin_link_5: geometry collision mesh filename=package://chin_crb7_description/meshes/collision/link_5.stl; visual mesh filename=package://chin_crb7_description/meshes/visual/link_5.dae
- link chin_link_6: geometry collision mesh filename=package://chin_crb7_description/meshes/collision/link_6.stl; visual mesh filename=package://chin_crb7_description/meshes/visual/link_6.dae

Commit message: refactor to xacro as interface

File: chin_crb7_description/urdf/chin_crb7.urdf.xacro (robot description, xacro)
@@ -1,169 +1,5 @@
 <?xml version="1.0"?>
 <robot name="chin_arm" xmlns:xacro="http://ros.org/wiki/xacro">
-  <xacro:property name="arm_id" value="chin"/>
-  <xacro:property name="arm_model" value="crb7"/>
-  <xacro:property name="description_pkg" value="${arm_id}_${arm_model}_description"/>
-  <xacro:property name="mesh" value="yes"/>
-  <!--is the robot being simulated in gazebo?-->
-  <xacro:property name="gazebo" value="false"/>
-  <xacro:property name="link_base_height" value="0.2038"/>
-  <xacro:property name="link_base_radius" value="0.095"/>
-  <xacro:property name="link_1_height" value="0.081"/>
-  <xacro:property name="link_1_radius" value="0.066"/>
-  <xacro:property name="link_2_height" value="0.082"/>
-  <xacro:property name="link_2_radius" value="0.066"/>
-  <xacro:property name="link_3_height" value="0.07"/>
-  <xacro:property name="link_3_radius" value="0.066"/>
-  <xacro:property name="link_4_height" value="0.398"/>
-  <xacro:property name="link_4_radius" value="0.055"/>
-  <xacro:property name="link_5_height" value="0.065"/>
-  <xacro:property name="link_5_radius" value="0.055"/>
-  <xacro:property name="link_6_height" value="0.063"/>
-  <xacro:property name="link_6_radius" value="0.055"/>
-  <xacro:property name="link_7_height" value="0.36"/>
-  <xacro:property name="link_7_radius" value="0.045"/>
-  <xacro:property name="link_8_height" value="0.083"/>
-  <xacro:property name="link_8_radius" value="0.045"/>
-  <xacro:property name="link_9_height" value="0.087"/>
-  <xacro:property name="link_9_radius" value="0.045"/>
-  <xacro:property name="link_10_height" value="0.083"/>
-  <xacro:property name="link_10_radius" value="0.045"/>
-  <xacro:property name="link_11_height" value="0.087"/>
-  <xacro:property name="link_11_radius" value="0.045"/>
-  <xacro:property name="link_12_height" value="0.083"/>
-  <xacro:property name="link_12_radius" value="0.045"/>
-  <xacro:property name="link_13_height" value="0.077"/>
-  <xacro:property name="link_13_radius" value="0.045"/>
-  <material name="white">
-    <color rgba="1 1 1 1"/>
-  </material>
-  <material name="blue">
-    <color rgba="0 0 0.8 1"/>
-  </material>
-  <material name="silver">
-    <color rgba="0.51 0.54 0.59 1"/>
-  </material>
-  <xacro:macro name="link_with_sc"  params="name link_height link_radius pos_xyz:='0 0 0' pos_rpy:='0 0 0' visual_color:='white' prefix=${arm_id} rpy:='0 0 0' **self_collision_geometries gazebo:=false">
-    <!--sub-link defining detailed meshes for collision with environment-->
-    <link name="${prefix}_${name}">
-      <visual>
-	      <origin xyz="${pos_xyz}" rpy="${pos_rpy}"/>
-        <geometry>
-          <!--the expression of condition cannot contain the key 'true/false' and '0/1'-->
-          <xacro:if value="${mesh == 'yes'}">
-            <mesh filename="package://${description_pkg}/meshes/visual/${name}.dae"/>
-          </xacro:if>
-          <xacro:unless value="${mesh == 'yes'}">
-            <cylinder length="${link_height}" radius="${link_radius}"/>
-          </xacro:unless>
-        </geometry>
-        <xacro:unless value="${mesh == 'yes'}">
-          <material name="${visual_color}"/>
-        </xacro:unless>
-      </visual>
-      <collision>
-	      <origin xyz="${pos_xyz}" rpy="${pos_rpy}"/>
-        <geometry>
-          <xacro:if value="${mesh == 'yes'}">
-            <mesh filename="package://${description_pkg}/meshes/collision/${name}.stl"/>
-          </xacro:if>
-          <xacro:unless value="${mesh == 'yes'}">
-            <cylinder length="${link_height}" radius="${link_radius}"/>
-          </xacro:unless>
-        </geometry>
-      </collision>
-      <xacro:if value="${gazebo}">
-        <xacro:inertial_props name="${name}"/>
-      </xacro:if>
-    </link>
-  </xacro:macro>
-  <!--fixed link0-->
-  <xacro:link_with_sc name="link_0" link_height="${link_base_height}" link_radius="${link_base_radius}" gazebo="${gazebo}">
-    <self_collision_geometries/>
-  </xacro:link_with_sc>
-  <!--link1 to link0-->
-  <xacro:link_with_sc name="link_1" link_height="${link_1_height}" link_radius="${link_1_radius}" pos_xyz="0 0 0" gazebo="${gazebo}">
-    <self_collision_geometries/>
-  </xacro:link_with_sc>
-  <joint name="${arm_id}_joint_1" type="revolute">
-    <safety_controller k_position="100.0" k_velocity="40.0" soft_lower_limit="${-pi}" soft_upper_limit="${pi}"/>
-    <origin rpy="0 0 0" xyz="0 0 ${link_base_height}"/>
-    <parent link="${arm_id}_link_0"/>
-    <child link="${arm_id}_link_1"/>
-    <axis xyz="0 0 1"/>
-    <limit lower="${-pi}" upper="${pi}" effort="0" velocity="0"/>
-    <dynamics D="1" K="7000" damping="0.003" friction="0.0" mu_coulomb="0" mu_viscous="16"/>
-  </joint>
-  <!--link2 to link1-->
-  <xacro:link_with_sc name="link_2" link_height="${link_2_height}" link_radius="${link_2_radius}" pos_xyz="0 0 0" gazebo="${gazebo}">
-    <self_collision_geometries/>
-  </xacro:link_with_sc>
-  <joint name="${arm_id}_joint_2" type="revolute">
-    <safety_controller k_position="100.0" k_velocity="40.0" soft_lower_limit="${-pi}" soft_upper_limit="${pi}"/>
-    <origin rpy="${-0.5*pi} 0 0" xyz="0 ${link_2_height} ${link_1_height}"/>
-    <parent link="${arm_id}_link_1"/>
-    <child link="${arm_id}_link_2"/>
-    <axis xyz="0 0 1"/>
-    <limit lower="${-pi}" upper="${pi}" effort="0" velocity="0"/>
-    <dynamics D="1" K="7000" damping="0.003" friction="0.0" mu_coulomb="0" mu_viscous="16"/>
-  </joint>
-  <!--link3 to link2-->
-  <xacro:link_with_sc name="link_3" link_height="${link_3_height}" link_radius="${link_3_radius}" pos_xyz="0 0 0" gazebo="${gazebo}">
-    <self_collision_geometries/>
-  </xacro:link_with_sc>
-  <joint name="${arm_id}_joint_3" type="revolute">
-    <safety_controller k_position="100.0" k_velocity="40.0" soft_lower_limit="${-160.0*pi/180.0}" soft_upper_limit="${160.0*pi/180.0}"/>
-    <origin rpy="${pi} 0 0" xyz="0 ${-link_4_height} 0"/>
-    <parent link="${arm_id}_link_2"/>
-    <child link="${arm_id}_link_3"/>
-    <axis xyz="0 0 1"/>
-    <limit lower="${-160.0*pi/180.0}" upper="${160.0*pi/180.0}" effort="0" velocity="0"/>
-    <dynamics D="1" K="7000" damping="0.003" friction="0.0" mu_coulomb="0" mu_viscous="16"/>
-  </joint>
-  <!--link4 to link3-->
-  <xacro:link_with_sc name="link_4" link_height="${link_4_height}" link_radius="${link_4_radius}" pos_xyz="0 0 0" gazebo="${gazebo}">
-    <self_collision_geometries/>
-  </xacro:link_with_sc>
-  <joint name="${arm_id}_joint_4" type="revolute">
-    <safety_controller k_position="100.0" k_velocity="40.0" soft_lower_limit="${-pi}" soft_upper_limit="${pi}"/>
-    <origin rpy="${pi} 0 0" xyz="0 ${link_7_height} ${-(link_8_height-link_6_height)}"/>
-    <parent link="${arm_id}_link_3"/>
-    <child link="${arm_id}_link_4"/>
-    <axis xyz="0 0 1"/>
-    <limit lower="${-pi}" upper="${pi}" effort="0" velocity="0"/>
-    <dynamics D="1" K="7000" damping="0.003" friction="0.0" mu_coulomb="0" mu_viscous="16"/>
-  </joint>
-  <!--link5 to link4-->
-  <xacro:link_with_sc name="link_5" link_height="${link_5_height}" link_radius="${link_5_radius}" pos_xyz="0 0 0" gazebo="${gazebo}">
-    <self_collision_geometries/>
-  </xacro:link_with_sc>
-  <joint name="${arm_id}_joint_5" type="revolute">
-    <safety_controller k_position="100.0" k_velocity="40.0" soft_lower_limit="${-pi}" soft_upper_limit="${pi}"/>
-    <origin rpy="${0.5*pi} 0 0" xyz="0 ${-link_10_height} ${link_11_height}"/>
-    <parent link="${arm_id}_link_4"/>
-    <child link="${arm_id}_link_5"/>
-    <axis xyz="0 0 1"/>
-    <limit lower="${-pi}" upper="${pi}" effort="0" velocity="0"/>
-    <dynamics D="1" K="7000" damping="0.003" friction="0.0" mu_coulomb="0" mu_viscous="16"/>
-  </joint>
-  <!--link6 to link5-->
-  <xacro:link_with_sc name="link_6" link_height="${link_6_height}" link_radius="${link_6_radius}" pos_xyz="0 0 0" gazebo="${gazebo}">
-    <self_collision_geometries/>
-  </xacro:link_with_sc>
-  <joint name="${arm_id}_joint_6" type="revolute">
-    <safety_controller k_position="100.0" k_velocity="40.0" soft_lower_limit="${-pi}" soft_upper_limit="${pi}"/>
-    <origin rpy="${-0.5*pi} 0 0" xyz="0 ${link_12_height} ${link_11_height}"/>
-    <parent link="${arm_id}_link_5"/>
-    <child link="${arm_id}_link_6"/>
-    <axis xyz="0 0 1"/>
-    <limit lower="${-pi}" upper="${pi}" effort="0" velocity="0"/>
-    <dynamics D="1" K="7000" damping="0.003" friction="0.0" mu_coulomb="0" mu_viscous="16"/>
-  </joint>
-  <!--link7 to link6-->
-  <link name="${arm_id}_link_7"/>
-  <joint name="${arm_id}_joint_7" type="fixed">
-    <origin rpy="0 0 ${-pi}" xyz="0 0 ${link_13_height}"/>
-    <parent link="${arm_id}_link_6"/>
-    <child link="${arm_id}_link_7"/>
-  </joint>
+  <xacro:include filename="$(find chin_crb7_description)/urdf/chin_arm.xacro"/>
+  <xacro:chin_arm arm_id="chin" model="crb7"/>
 </robot>
