Commit message: add link7 to group

File: chin_crb7_description/urdf/chin_arm.xacro (robot description, xacro)
@@ -138,5 +138,5 @@
     <link name="${arm_id}_link_7"/>
     <joint name="${arm_id}_joint_7" type="fixed">
-      <origin rpy="0 0 ${-pi}" xyz="0 0 ${link_13_height}"/>
+      <origin rpy="0 0 0" xyz="0 0 ${link_13_height}"/>
       <parent link="${arm_id}_link_6"/>
       <child link="${arm_id}_link_7"/>

File: chin_crb7_moveit_config/config/gazebo_chin_arm.urdf (robot description, URDF)
Before this commit: robot chin_arm, 8 links, 7 joints
Joints:
- joint chin_joint_3: limit lower=-2.7925 upper=2.7925 effort=0 velocity=0 -> lower=-2.79252680319 upper=2.79252680319 effort=0 velocity=0

Commit message: change name to tcp

File: chin_crb7_description/urdf/chin_arm.xacro (robot description, xacro)
@@ -136,9 +136,9 @@
     </joint>
     <!--link7 to link6-->
-    <link name="${arm_id}_link_7"/>
-    <joint name="${arm_id}_joint_7" type="fixed">
-      <origin rpy="0 0 0" xyz="0 0 ${link_13_height}"/>
+    <link name="${arm_id}_link_tcp"/>
+    <joint name="${arm_id}_joint_tcp" type="fixed">
+      <origin rpy="${pi} 0 ${-0.5 * pi}" xyz="0 0 ${link_13_height}"/>
       <parent link="${arm_id}_link_6"/>
-      <child link="${arm_id}_link_7"/>
+      <child link="${arm_id}_link_tcp"/>
     </joint>
   </xacro:macro>

File: chin_crb7_moveit_config/config/gazebo_chin_arm.urdf (robot description, URDF)
Before this commit: robot chin_arm, 8 links, 7 joints
Links:
- removed link chin_link_7
- added link chin_link_tcp
Joints:
- removed joint chin_joint_7
- added joint chin_joint_tcp: type fixed, parent chin_link_6, child chin_link_tcp, origin xyz=0 0 0.077 rpy=3.14159265359 0 -1.57079632679
